Commit message: Add Bittle head with a working neck joint (servo 0)
Head, jaw, neck mount and neck servo meshes from Petoi's official model
(PetoiCamp/ros_opencat, MIT), fitted via the four shoulder hinges and
turned so neck angle 0 faces forward. neck-joint (+-90 deg, positive =
left) defaults to OpenCat servo 0, so skills and I packets drive the
real head. Unedited older bundled models in saved projects upgrade
automatically; saved servo mappings gain the new joint. Stage shows
the actual joint count.

Co-Authored-By: Claude Opus 5.5 <noreply@anthropic.com>

File: app/tests/fixtures/bittle-headless.urdf (robot description, URDF)
Before this commit: robot bittle, 15 links, 14 joints
Links:
- removed link head-link
- removed link neck-mount-link
Joints:
- removed joint neck-joint
- removed joint neck-mount-joint
