Commit message: Fix simulated skills (sit, behaviour timing), start in zero pose, tidy inspector
- Leg joint limits are mirror-symmetric and cover Petoi's skills
  (shoulders +-125, knees -80..125 in servo terms), so sit reaches 105
  on both sides. Projects with the previous bundled model upgrade.
- Behaviour timing follows the firmware's transform() (steps of ~8 ms,
  cosine easing, delay x 50 ms), capped at a realistic 350 deg/s servo
  speed; goodbye, hug, cheer and nod no longer run too fast.
- The Studio starts with every robot in the zero pose.
- The inspector is just Robot control; Object and Robot+ properties
  appear under the Stage for the selected item; the duplicate Model
  URDF tab is removed (the Robot Editor has it).

Co-Authored-By: Claude Opus 5.5 <noreply@anthropic.com>

File: app/tests/fixtures/bittle-narrow-limits.urdf (robot description, URDF)
Before this commit: robot bittle, 15 links, 14 joints
Joints:
- joint left-back-knee-joint: limit lower=-1.39626 upper=2.18166 effort=1.0 velocity=1.5708 -> lower=-1.22173 upper=1.48353 effort=1.0 velocity=1.5708
- joint left-back-shoulder-joint: limit lower=-2.18166 upper=2.18166 effort=1.0 velocity=1.5708 -> lower=-1.5708 upper=1.22173 effort=1.0 velocity=1.5708
- joint left-front-knee-joint: limit lower=-1.39626 upper=2.18166 effort=1.0 velocity=1.5708 -> lower=-1.22173 upper=1.48353 effort=1.0 velocity=1.5708
- joint left-front-shoulder-joint: limit lower=-2.18166 upper=2.18166 effort=1.0 velocity=1.5708 -> lower=-1.5708 upper=1.22173 effort=1.0 velocity=1.5708
- joint right-back-knee-joint: limit lower=-2.18166 upper=1.39626 effort=1.0 velocity=1.5708 -> lower=-1.22173 upper=1.48353 effort=1.0 velocity=1.5708
- joint right-back-shoulder-joint: limit lower=-2.18166 upper=2.18166 effort=1.0 velocity=1.5708 -> lower=-1.5708 upper=1.22173 effort=1.0 velocity=1.5708
- joint right-front-knee-joint: limit lower=-2.18166 upper=1.39626 effort=1.0 velocity=1.5708 -> lower=-1.22173 upper=1.48353 effort=1.0 velocity=1.5708
- joint right-front-shoulder-joint: limit lower=-2.18166 upper=2.18166 effort=1.0 velocity=1.5708 -> lower=-1.5708 upper=1.22173 effort=1.0 velocity=1.5708
